File: 4xTCAN4550-HAT.sch (KiCad schematic (older format))
At the start: 14 parts, among them J1 Conn_02x04_Odd_Even, U1 LM27313XMF, X1 ASV-40.000MHz

Commit message: remove rst, add wake and is_awake
Connections:
- wire segments 125 -> 114
- no-connect marks 1 -> 2
Other:
- moved on the sheet: U1
