File: TCAN4550.sch (KiCad schematic (older format))
At the start: 11 parts, among them U3 TCAN4550

Commit message: remove rst, add wake and is_awake
Parts:
- added Q1: 2N7002, Package_TO_SOT_SMD:SOT-23, symbol Transistor_FET:2N7002
- added R26, R27, R29: 10K, Resistor_SMD:R_0603_1608Metric, symbol Device:R_Small
- added R28: 5K6, Resistor_SMD:R_0603_1608Metric, symbol Device:R_Small
Connections:
- net labels added: IS_AWAKE, WAKE
- net labels removed: RST
- wire segments 31 -> 42
- no-connect marks 4 -> 5

Commit message: move wake fet pull-ups from transceivers to raspi-hat schematic page
Parts:
- removed R26: 10K, Resistor_SMD:R_0603_1608Metric, symbol Device:R_Small
- C7: value 330nF -> 1uF
Connections:
- wire segments 42 -> 40
Changed lines of the file:
@@
 AR Path="/5C990443/5C960A4F" Ref="#PWR048"  Part="1"
 AR Path="/5C9AD914/5C960A4F" Ref="#PWR061"  Part="1"
-F 0 "#PWR061" H 5550 2900 50  0001 C CNN
+F 0 "#PWR022" H 5550 2900 50  0001 C CNN
 F 1 "+3V3" H 5565 3223 50  0000 C CNN
 F 2 "" H 5550 3050 50  0001 C CNN
@@
 AR Path="/5C990443/5C960A5C" Ref="#PWR052"  Part="1"
 AR Path="/5C9AD914/5C960A5C" Ref="#PWR065"  Part="1"
-F 0 "#PWR065" H 6500 3050 50  0001 C CNN
+F 0 "#PWR026" H 6500 3050 50  0001 C CNN
 F 1 "+3V3" H 6515 3373 50  0000 C CNN
 F 2 "" H 6500 3200 50  0001 C CNN
@@
 AR Path="/5C990443/5C960A62" Ref="#PWR053"  Part="1"
 AR Path="/5C9AD914/5C960A62" Ref="#PWR066"  Part="1"
-F 0 "#PWR066" H 6500 3150 50  0001 C CNN
+F 0 "#PWR027" H 6500 3150 50  0001 C CNN
 F 1 "GND" H 6505 3227 50  0000 C CNN
 F 2 "" H 6500 3400 50  0001 C CNN
@@
 AR Path="/5C990443/5C960A68" Ref="#PWR049"  Part="1"
 AR Path="/5C9AD914/5C960A68" Ref="#PWR062"  Part="1"
-F 0 "#PWR062" H 5650 4800 50  0001 C CNN
+F 0 "#PWR023" H 5650 4800 50  0001 C CNN
 F 1 "GND" H 5655 4877 50  0000 C CNN
 F 2 "" H 5650 5050 50  0001 C CNN
@@
 AR Path="/5C990443/5C960A76" Ref="#PWR056"  Part="1"
 AR Path="/5C9AD914/5C960A76" Ref="#PWR069"  Part="1"
-F 0 "#PWR069" H 6950 3150 50  0001 C CNN
+F 0 "#PWR030" H 6950 3150 50  0001 C CNN
 F 1 "GND" H 6955 3227 50  0000 C CNN
 F 2 "" H 6950 3400 50  0001 C CNN
@@
 AR Path="/5C990443/5C960A89" Ref="#PWR058"  Part="1"
 AR Path="/5C9AD914/5C960A89" Ref="#PWR071"  Part="1"
-F 0 "#PWR071" H 7350 3150 50  0001 C CNN
+F 0 "#PWR032" H 7350 3150 50  0001 C CNN
 F 1 "GND" H 7355 3227 50  0000 C CNN
 F 2 "" H 7350 3400 50  0001 C CNN
@@
 AR Path="/5C9AD914/5C960AA9" Ref="C22"  Part="1"
 F 0 "C7" H 7192 4646 50  0000 L CNN
-F 1 "330nF" H 7192 4555 50  0000 L CNN
+F 1 "1uF" H 7192 4555 50  0000 L CNN
 F 2 "Capacitor_SMD:C_0603_1608Metric" H 7100 4600 50  0001 C CNN
 F 3 "~" H 7100 4600 50  0001 C CNN
@@
 AR Path="/5C990443/5C960AB0" Ref="#PWR054"  Part="1"
 AR Path="/5C9AD914/5C960AB0" Ref="#PWR067"  Part="1"
-F 0 "#PWR067" H 7100 4450 50  0001 C CNN
+F 0 "#PWR028" H 7100 4450 50  0001 C CNN
 F 1 "GND" H 7105 4527 50  0000 C CNN
 F 2 "" H 7100 4700 50  0001 C CNN
@@
 AR Path="/5C990443/5C960AED" Ref="#PWR046"  Part="1"
 AR Path="/5C9AD914/5C960AED" Ref="#PWR059"  Part="1"
-F 0 "#PWR059" H 5100 4450 50  0001 C CNN
+F 0 "#PWR020" H 5100 4450 50  0001 C CNN
 F 1 "GND" H 5000 4700 50  0000 C CNN
 F 2 "" H 5100 4700 50  0001 C CNN
@@
 AR Path="/5C990443/5C77F66E" Ref="#PWR0103"  Part="1"
 AR Path="/5C9AD914/5C77F66E" Ref="#PWR0104"  Part="1"
-F 0 "#PWR0104" H 5750 2900 50  0001 C CNN
+F 0 "#PWR0101" H 5750 2900 50  0001 C CNN
 F 1 "VCC" H 5767 3223 50  0000 C CNN
 F 2 "" H 5750 3050 50  0001 C CNN
@@
 AR Path="/5C990443/5C77F9AF" Ref="#PWR0109"  Part="1"
 AR Path="/5C9AD914/5C77F9AF" Ref="#PWR0111"  Part="1"
-F 0 "#PWR0111" H 6950 3050 50  0001 C CNN
+F 0 "#PWR0105" H 6950 3050 50  0001 C CNN
 F 1 "VCC" H 6967 3373 50  0000 C CNN
 F 2 "" H 6950 3200 50  0001 C CNN
@@
 AR Path="/5C990443/5C77FB3D" Ref="#PWR0110"  Part="1"
 AR Path="/5C9AD914/5C77FB3D" Ref="#PWR0112"  Part="1"
-F 0 "#PWR0112" H 7350 3050 50  0001 C CNN
+F 0 "#PWR0106" H 7350 3050 50  0001 C CNN
 F 1 "VCC" H 7367 3373 50  0000 C CNN
 F 2 "" H 7350 3200 50  0001 C CNN
@@
 AR Path="/5C990443/5C78747F" Ref="#PWR0117"  Part="1"
 AR Path="/5C9AD914/5C78747F" Ref="#PWR0118"  Part="1"
-F 0 "#PWR0118" H 4750 3150 50  0001 C CNN
+F 0 "#PWR0115" H 4750 3150 50  0001 C CNN
 F 1 "+3V3" H 4765 3473 50  0000 C CNN
 F 2 "" H 4750 3300 50  0001 C CNN
@@
 AR Path="/5C990443/5C7820A4" Ref="#PWR031"  Part="1"
 AR Path="/5C9AD914/5C7820A4" Ref="#PWR037"  Part="1"
-F 0 "#PWR037" H 7500 3850 50  0001 C CNN
+F 0 "#PWR024" H 7500 3850 50  0001 C CNN
 F 1 "GND" V 7505 3972 50  0000 R CNN
 F 2 "" H 7500 4100 50  0001 C CNN
@@
 AR Path="/5C990443/5C7810EA" Ref="#PWR0121"  Part="1"
 AR Path="/5C9AD914/5C7810EA" Ref="#PWR0122"  Part="1"
-F 0 "#PWR0122" H 4250 3950 50  0001 C CNN
+F 0 "#PWR0119" H 4250 3950 50  0001 C CNN
 F 1 "+3V3" H 4265 4273 50  0000 C CNN
 F 2 "" H 4250 4100 50  0001 C CNN
@@
 AR Path="/5C990443/5C7E8484" Ref="#PWR063"  Part="1"
 AR Path="/5C9AD914/5C7E8484" Ref="#PWR073"  Part="1"
-F 0 "#PWR073" H 4650 5050 50  0001 C CNN
+F 0 "#PWR034" H 4650 5050 50  0001 C CNN
 F 1 "GND" H 4655 5127 50  0000 C CNN
 F 2 "" H 4650 5300 50  0001 C CNN
@@
 AR Path="/5C990443/5C7E8DCC" Ref="#PWR060"  Part="1"
 AR Path="/5C9AD914/5C7E8DCC" Ref="#PWR072"  Part="1"
-F 0 "#PWR072" H 4650 4450 50  0001 C CNN
+F 0 "#PWR025" H 4650 4450 50  0001 C CNN
 F 1 "VCC" H 4550 4700 50  0000 C CNN
 F 2 "" H 4650 4600 50  0001 C CNN
@@
 Wire Wire Line
 	4650 4850 4650 4900
-$Comp
-L Device:R_Small R?
-U 1 1 5C7EA4FF
-P 4300 4900
-AR Path="/5C7EA4FF" Ref="R?"  Part="1"
-AR Path="/5C960736/5C7EA4FF" Ref="R26"  Part="1"
-AR Path="/5C970AFF/5C7EA4FF" Ref="R30"  Part="1"
-AR Path="/5C990443/5C7EA4FF" Ref="R34"  Part="1"
-AR Path="/5C9AD914/5C7EA4FF" Ref="R38"  Part="1"
-F 0 "R26" V 4200 4900 50  0000 C CNN
-F 1 "10K" V 4400 4900 50  0000 C CNN
-F 2 "Resistor_SMD:R_0603_1608Metric" H 4300 4900 50  0001 C CNN
-F 3 "~" H 4300 4900 50  0001 C CNN
-	1    4300 4900
-	1    0    0    -1
-$EndComp
-$Comp
-L power:+3V3 #PWR?
-U 1 1 5C7EA505
-P 4300 4800
-AR Path="/5C7EA505" Ref="#PWR?"  Part="1"
-AR Path="/5C960736/5C7EA505" Ref="#PWR021"  Part="1"
-AR Path="/5C970AFF/5C7EA505" Ref="#PWR044"  Part="1"
-AR Path="/5C990443/5C7EA505" Ref="#PWR057"  Part="1"
-AR Path="/5C9AD914/5C7EA505" Ref="#PWR070"  Part="1"
-F 0 "#PWR070" H 4300 4650 50  0001 C CNN
-F 1 "+3V3" H 4315 4973 50  0000 C CNN
-F 2 "" H 4300 4800 50  0001 C CNN
-F 3 "" H 4300 4800 50  0001 C CNN
-	1    4300 4800
-	1    0    0    -1
-$EndComp
 Text HLabel 4100 5100 0    50   Input ~ 0
 WAKE
-Wire Wire Line
-	4300 5000 4300 5100
-Connection ~ 4300 5100
-Wire Wire Line
-	4300 5100 4350 5100
-Wire Wire Line
-	4100 5100 4300 5100
 Wire Wire Line
 	4750 3550 5150 3550
@@
 AR Path="/5C990443/5C7FCC02" Ref="#PWR064"  Part="1"
 AR Path="/5C9AD914/5C7FCC02" Ref="#PWR074"  Part="1"
-F 0 "#PWR074" H 6350 4650 50  0001 C CNN
+F 0 "#PWR038" H 6350 4650 50  0001 C CNN
 F 1 "GND" H 6355 4727 50  0000 C CNN
 F 2 "" H 6350 4900 50  0001 C CNN
@@
 AR Path="/5C990443/5C7FE182" Ref="#PWR068"  Part="1"
 AR Path="/5C9AD914/5C7FE182" Ref="#PWR075"  Part="1"
-F 0 "#PWR075" H 6850 5200 50  0001 C CNN
+F 0 "#PWR042" H 6850 5200 50  0001 C CNN
 F 1 "GND" H 6855 5277 50  0000 C CNN
 F 2 "" H 6850 5450 50  0001 C CNN
@@
 	6150 4650 6350 4650
 NoConn ~ 5150 3350
+Wire Wire Line
+	4100 5100 4350 5100
 $EndSCHEMATC
