File: raspi-hat.sch (KiCad schematic (older format))
At the start: 9 parts, among them J2 Raspberry_Pi_2_3, U2 AT24CS64-MAHM

Commit message: fix eeprom
Changed lines of the file:
@@
 U 1 1 5C75DA44
 P 7450 3250
-F 0 "U2" H 7200 3500 50  0000 C CNN
-F 1 "AT24CS64-MAHM" H 7800 3500 50  0000 C CNN
+F 0 "U2" H 7700 3500 50  0000 C CNN
+F 1 "AT24CS64-MAHM" H 7450 2950 50  0000 C CNN
 F 2 "Package_DFN_QFN:DFN-8-1EP_3x2mm_P0.5mm_EP1.3x1.5mm" H 7450 3250 50  0001 C CNN
 F 3 "http://ww1.microchip.com/downloads/en/DeviceDoc/Atmel-8870-SEEPROM-AT24CS64-Datasheet.pdf" H 7450 3250 50  0001 C CNN
 	1    7450 3250
-	1    0    0    -1
+	-1   0    0    -1
 $EndComp
 $EndSCHEMATC

Commit message: remove rst, add wake and is_awake
Connections:
- net labels added: CAN0_IS_AWAKE, CAN0_WAKE, CAN1_IS_AWAKE, CAN1_WAKE, CAN2_IS_AWAKE, CAN2_WAKE, CAN3_IS_AWAKE, CAN3_WAKE
- net labels removed: CAN0_RST, CAN1_RST, CAN2_RST, CAN3_RST
- no-connect marks 8 -> 4
Changed lines of the file:
@@
 L Device:R_Small R?
 U 1 1 5C9248F9
-P 6600 4350
+P 6850 4350
 AR Path="/5C9248F9" Ref="R?"  Part="1"
 AR Path="/5C921E3E/5C9248F9" Ref="R8"  Part="1"
-F 0 "R8" V 6500 4350 50  0000 C CNN
-F 1 "56R" V 6700 4350 50  0000 C CNN
-F 2 "Resistor_SMD:R_0603_1608Metric" H 6600 4350 50  0001 C CNN
-F 3 "~" H 6600 4350 50  0001 C CNN
-	1    6600 4350
+F 0 "R8" V 6750 4350 50  0000 C CNN
+F 1 "56R" V 6950 4350 50  0000 C CNN
+F 2 "Resistor_SMD:R_0603_1608Metric" H 6850 4350 50  0001 C CNN
+F 3 "~" H 6850 4350 50  0001 C CNN
+	1    6850 4350
 	0    1    1    0
 $EndComp
@@
 L Device:R_Small R?
 U 1 1 5C924900
-P 6600 4650
+P 6850 4650
 AR Path="/5C924900" Ref="R?"  Part="1"
 AR Path="/5C921E3E/5C924900" Ref="R9"  Part="1"
-F 0 "R9" V 6500 4650 50  0000 C CNN
-F 1 "56R" V 6700 4650 50  0000 C CNN
-F 2 "Resistor_SMD:R_0603_1608Metric" H 6600 4650 50  0001 C CNN
-F 3 "~" H 6600 4650 50  0001 C CNN
-	1    6600 4650
+F 0 "R9" V 6750 4650 50  0000 C CNN
+F 1 "56R" V 6950 4650 50  0000 C CNN
+F 2 "Resistor_SMD:R_0603_1608Metric" H 6850 4650 50  0001 C CNN
+F 3 "~" H 6850 4650 50  0001 C CNN
+	1    6850 4650
 	0    1    1    0
 $EndComp
@@
 Text HLabel 5950 4350 2    50   Input ~ 0
 SPI0_MISO
-Text HLabel 6700 4350 2    50   Output ~ 0
+Text HLabel 6950 4350 2    50   Output ~ 0
 SPI0_MOSI
-Text HLabel 6700 4650 2    50   Output ~ 0
+Text HLabel 6950 4650 2    50   Output ~ 0
 SPI0_SCK
 Wire Wire Line
 	3800 3850 3850 3850
 Wire Wire Line
-	3850 3850 3850 3950
-Wire Wire Line
 	3850 3950 4350 3950
 Wire Wire Line
-	3850 4050 3850 4150
-Wire Wire Line
 	3850 4150 3800 4150
 Wire Wire Line
 	3850 4050 4350 4050
 Wire Wire Line
-	6450 4450 6450 4350
-Wire Wire Line
-	6450 4350 6500 4350
-Wire Wire Line
-	5950 4450 6450 4450
-Wire Wire Line
-	6450 4550 6450 4650
-Wire Wire Line
-	6450 4650 6500 4650
-Wire Wire Line
-	5950 4550 6450 4550
-Text HLabel 4350 4450 0    50   Output ~ 0
-CAN0_RST
-Text HLabel 4350 4550 0    50   Input ~ 0
+	6700 4450 6700 4350
+Wire Wire Line
+	6700 4350 6750 4350
+Wire Wire Line
+	6700 4550 6700 4650
+Wire Wire Line
+	6700 4650 6750 4650
+Text HLabel 4350 4750 0    50   Input ~ 0
 CAN0_INT
-Text HLabel 5950 3850 2    50   Output ~ 0
-CAN1_RST
-Text HLabel 5950 3950 2    50   Input ~ 0
+Text HLabel 4350 4450 0    50   Input ~ 0
 CAN1_INT
-Text HLabel 5950 4750 2    50   Output ~ 0
-CAN2_RST
-Text HLabel 5950 4850 2    50   Input ~ 0
+Text HLabel 5950 3850 2    50   Input ~ 0
 CAN2_INT
-Text HLabel 4350 4650 0    50   Output ~ 0
-CAN3_RST
-Text HLabel 4350 3450 0    50   Input ~ 0
+Text HLabel 5950 4750 2    50   Input ~ 0
 CAN3_INT
-NoConn ~ 4350 3150
-NoConn ~ 4350 3250
-NoConn ~ 4350 4250
-NoConn ~ 4350 4350
-NoConn ~ 4350 4750
-NoConn ~ 5950 3450
-NoConn ~ 5950 3550
-NoConn ~ 5950 3750
 Wire Wire Line
 	6950 3550 6950 3350
 Wire Wire Line
 	6950 3350 7050 3350
-Wire Wire Line
-	5950 3250 6600 3250
 Wire Wire Line
 	5950 3150 6350 3150
@@
 L power:+3V3 #PWR?
 U 1 1 5C780CCA
-P 8250 3100
+P 8200 3350
 AR Path="/5C780CCA" Ref="#PWR?"  Part="1"
 AR Path="/5C921E3E/5C780CCA" Ref="#PWR0113"  Part="1"
-F 0 "#PWR0113" H 8250 2950 50  0001 C CNN
-F 1 "+3V3" H 8265 3273 50  0000 C CNN
-F 2 "" H 8250 3100 50  0001 C CNN
-F 3 "" H 8250 3100 50  0001 C CNN
-	1    8250 3100
+F 0 "#PWR0113" H 8200 3200 50  0001 C CNN
+F 1 "+3V3" H 8215 3523 50  0000 C CNN
+F 2 "" H 8200 3350 50  0001 C CNN
+F 3 "" H 8200 3350 50  0001 C CNN
+	1    8200 3350
 	1    0    0    -1
 $EndComp
@@
 L power:GND #PWR?
 U 1 1 5C781767
-P 8250 3300
+P 8200 3550
 AR Path="/5C781767" Ref="#PWR?"  Part="1"
 AR Path="/5C921E3E/5C781767" Ref="#PWR0114"  Part="1"
-F 0 "#PWR0114" H 8250 3050 50  0001 C CNN
-F 1 "GND" H 8255 3127 50  0000 C CNN
-F 2 "" H 8250 3300 50  0001 C CNN
-F 3 "" H 8250 3300 50  0001 C CNN
-	1    8250 3300
+F 0 "#PWR0114" H 8200 3300 50  0001 C CNN
+F 1 "GND" H 8205 3377 50  0000 C CNN
+F 2 "" H 8200 3550 50  0001 C CNN
+F 3 "" H 8200 3550 50  0001 C CNN
+	1    8200 3550
 	1    0    0    -1
 $EndComp
@@
 L Device:C_Small C25
 U 1 1 5C780C94
-P 8250 3200
-F 0 "C25" H 8342 3246 50  0000 L CNN
-F 1 "100nF" H 8342 3155 50  0000 L CNN
-F 2 "Capacitor_SMD:C_0603_1608Metric" H 8250 3200 50  0001 C CNN
-F 3 "~" H 8250 3200 50  0001 C CNN
-	1    8250 3200
+P 8200 3450
+F 0 "C25" H 8292 3496 50  0000 L CNN
+F 1 "100nF" H 8292 3405 50  0000 L CNN
+F 2 "Capacitor_SMD:C_0603_1608Metric" H 8200 3450 50  0001 C CNN
+F 3 "~" H 8200 3450 50  0001 C CNN
+	1    8200 3450
 	1    0    0    -1
 $EndComp
@@
 P 7450 3250
 F 0 "U2" H 7700 3500 50  0000 C CNN
-F 1 "AT24CS64-MAHM" H 7450 2950 50  0000 C CNN
+F 1 "AT24CS64-MAHM" H 7100 3500 50  0000 C CNN
 F 2 "Package_DFN_QFN:DFN-8-1EP_3x2mm_P0.5mm_EP1.3x1.5mm" H 7450 3250 50  0001 C CNN
 F 3 "http://ww1.microchip.com/downloads/en/DeviceDoc/Atmel-8870-SEEPROM-AT24CS64-Datasheet.pdf" H 7450 3250 50  0001 C CNN
@@
 	-1   0    0    -1
 $EndComp
+Text HLabel 5950 3450 2    50   Output ~ 0
+CAN0_WAKE
+Text HLabel 5950 3550 2    50   Output ~ 0
+CAN1_WAKE
+Text HLabel 4350 3450 0    50   Output ~ 0
+CAN2_WAKE
+Text HLabel 4350 4650 0    50   Output ~ 0
+CAN3_WAKE
+Text HLabel 5950 3750 2    50   Input ~ 0
+CAN0_IS_AWAKE
+Text HLabel 4350 4550 0    50   Input ~ 0
+CAN1_IS_AWAKE
+Text HLabel 5950 3950 2    50   Input ~ 0
+CAN2_IS_AWAKE
+Text HLabel 5950 4850 2    50   Input ~ 0
+CAN3_IS_AWAKE
+Wire Wire Line
+	3850 4050 3850 4150
+Wire Wire Line
+	3850 3850 3850 3950
+Wire Wire Line
+	5950 3250 6600 3250
+Wire Wire Line
+	5950 4450 6700 4450
+Wire Wire Line
+	5950 4550 6700 4550
+NoConn ~ 4350 3250
+NoConn ~ 4350 4250
+NoConn ~ 4350 3150
+NoConn ~ 4350 4350
 $EndSCHEMATC

Commit message: move wake fet pull-ups from transceivers to raspi-hat schematic page
Parts:
- added R26, R30, R34, R38: 10K, Resistor_SMD:R_0603_1608Metric, symbol Device:R_Small
Connections:
- wire segments 54 -> 70
Other:
- moved on the sheet: U2
